File: 79 Board/79 Board.sch (KiCad schematic (older format))
At the start: 31 parts, among them T1 TEST_HOLE, T2 TEST_HOLE, T3 TEST_HOLE, T4 TEST_HOLE

Commit message: finished 79 and myDaq, started mtb
Parts:
- removed C1, C5: 0.1µF, symbol C
- removed C2, C6: 1.0µF, symbol C
- removed MB_CONN1: CONN_02X07, symbol MB_CONN
- removed OPAMP1: MCP6002, symbol MCP6002
- added OPAMP1: MCP6002_flip, symbol MCP6002_flip
- added U?: MB_CONN, symbol MB_CONN
- 4x1_A1, 4x1_B1: footprint (none) -> MCB_footprints:Molex_Picoflex_Header_903250004
- C1: renamed from C3; footprint (none) -> MCB_footprints:Standard_Capacitor
- C2: renamed from C4; footprint (none) -> MCB_footprints:Standard_Capacitor
- C3: renamed from C7; footprint (none) -> MCB_footprints:Standard_Capacitor
- C4: renamed from C8; footprint (none) -> MCB_footprints:Standard_Capacitor
- C5: renamed from C9; footprint (none) -> MCB_footprints:Standard_Capacitor
- C6: renamed from C10; footprint (none) -> MCB_footprints:Standard_Capacitor
- HBRIDGE1, HBRIDGE2: footprint (none) -> Housings_DIP:DIP-16_W7.62mm_Socket
- JP1, JP2: footprint (none) -> Pin_Headers:Pin_Header_Angled_2x02_Pitch2.54mm
- PRES1: footprint (none) -> Pin_Headers:Pin_Header_Angled_1x06_Pitch2.54mm
- P_OUT1, T_OUT1: footprint (none) -> MCB_footprints:TESTPOINT_SMALL
- R1, R2, R5: footprint (none) -> Resistors_THT:R_Axial_DIN0207_L6.3mm_D2.5mm_P7.62mm_Horizontal
- R3: renamed from R4; footprint (none) -> Resistors_THT:R_Axial_DIN0207_L6.3mm_D2.5mm_P7.62mm_Horizontal
- R4: renamed from R3; footprint (none) -> Resistors_THT:R_Axial_DIN0207_L6.3mm_D2.5mm_P7.62mm_Horizontal
- T1, T2, T3, T4: footprint (none) -> MCB_footprints:TESTPOINT_LARGE
- TEMP1: footprint (none) -> Pin_Headers:Pin_Header_Angled_1x02_Pitch2.54mm
Connections:
- net +5V: now also OPAMP1.8 (Vdd), U?.12 (5V)
- net 1A: now also HBRIDGE1.10 (3A), U?.11 (1A); no longer HBRIDGE1.15 (4A)
- net 1Y: now also HBRIDGE1.11 (3Y); no longer HBRIDGE1.14 (4Y)
- net 2A: now also HBRIDGE1.15 (4A), U?.4 (2A); no longer HBRIDGE1.10 (3A)
- net 2Y: now also HBRIDGE1.14 (4Y), JP1.2 (P2); no longer HBRIDGE1.11 (3Y), JP1.3 (P3)
- net 3A: now also HBRIDGE1.7 (2A), U?.10 (3A); no longer HBRIDGE1.3 (1Y)
- net 3Y: now also HBRIDGE1.6 (2Y), JP1.3 (P3); no longer HBRIDGE1.2 (1A), JP1.2 (P2)
- net 4A: now also HBRIDGE1.2 (1A), U?.5 (4A); no longer HBRIDGE1.6 (2Y)
- net 4Y: now also HBRIDGE1.3 (1Y); no longer HBRIDGE1.7 (2A)
- net 5A: now also HBRIDGE2.10 (3A), U?.9 (5A); no longer HBRIDGE2.15 (4A)
- net 5Y: now also HBRIDGE2.11 (3Y); no longer HBRIDGE2.14 (4Y)
- net 6A: now also HBRIDGE2.15 (4A), U?.6 (6A); no longer HBRIDGE2.10 (3A)
- net 6Y: now also HBRIDGE2.14 (4Y), JP2.2 (P2); no longer HBRIDGE2.11 (3Y), JP2.3 (P3)
- net 7A: now also HBRIDGE2.7 (2A), U?.8 (7A); no longer HBRIDGE2.3 (1Y)
- net 7Y: now also HBRIDGE2.6 (2Y), JP2.3 (P3); no longer HBRIDGE2.2 (1A), JP2.2 (P2)
- net 8A: now also HBRIDGE2.2 (1A), U?.7 (8A); no longer HBRIDGE2.6 (2Y)
- net 8Y: now also HBRIDGE2.3 (1Y); no longer HBRIDGE2.7 (2A)
- net AGND: now also OPAMP1.4 (Vss), U?.14 (AGND)
- net Earth: now also U?.1 (GND)
- net PRES: now also OPAMP1.7 (VoutB), U?.2 (PRES)
- net TEMP: now also OPAMP1.1 (VoutA), OPAMP1.2 (VinA-), U?.13 (TEMP)
- net Vm: now also U?.3 (Vm)
- net at PRES1.1 (Vout), P_OUT1.1: now also OPAMP1.5 (VinB+)
- net at R2.1, R3.1, R4.2: now also OPAMP1.6 (VinB-)
- net at R5.2, TEMP1.2, T_OUT1.1: now also OPAMP1.3 (VinA+)
