File: myDAQ Breakout Board/myDAQ Breakout Board.kicad_pcb (KiCad board)
At the start: 2 copper layers, 31.5 x 64 mm, 16 parts

Commit message: finished 79 and myDaq, started mtb
Routing:
- removed copper zone on F.Cu, net GND
Changed lines of the file:
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@@
 (kicad_pcb (version 4) (host pcbnew 4.0.6)
   (general
-    (links 54)
+    (links 55)
     (no_connects 0)
     (area 175.124999 85.525 215.975001 152.983001)
@@
     )
   )
-  (module MDB_footprints:7805-thermal-conn (layer F.Cu)
-    (at 193.04 105.41 180)
-    (fp_text reference VREG (at 0 2.6 180) (layer F.SilkS)
-      (effects (font (size 1.2 1.2) (thickness 0.15)))
-    )
-    (fp_text value 7805 (at 0 -20.32 180) (layer F.Fab)
-      (effects (font (size 1.2 1.2) (thickness 0.15)))
-    )
-    (fp_line (start 3.94 -1.4) (end -3.94 -1.4) (layer F.SilkS) (width 0.15))
-    (fp_line (start -3.94 -19) (end 3.94 -19) (layer F.SilkS) (width 0.15))
-    (fp_line (start 3.94 -19) (end 3.94 1.4) (layer F.SilkS) (width 0.15))
-    (fp_line (start 3.94 1.4) (end -3.94 1.4) (layer F.SilkS) (width 0.15))
-    (fp_line (start -3.94 1.4) (end -3.94 -19) (layer F.SilkS) (width 0.15))
-    (fp_line (start -1.27 -1.4) (end -1.27 1.4) (layer F.SilkS) (width 0.15))
-    (pad 2 thru_hole circle (at -3.175 -13.335 180) (size 0.6 0.6) (drill 0.33) (layers *.Cu *.Mask)
-      (net 3 GND) (zone_connect 1))
-    (pad 2 thru_hole circle (at -3.175 -14.605 180) (size 0.6 0.6) (drill 0.33) (layers *.Cu *.Mask)
-      (net 3 GND) (zone_connect 1))
-    (pad 2 thru_hole circle (at -3.175 -15.875 180) (size 0.6 0.6) (drill 0.33) (layers *.Cu *.Mask)
-      (net 3 GND) (zone_connect 1))
-    (pad 2 thru_hole circle (at -3.175 -17.145 180) (size 0.6 0.6) (drill 0.33) (layers *.Cu *.Mask)
-      (net 3 GND) (zone_connect 1))
-    (pad 2 thru_hole circle (at -2.54 -18.415 180) (size 0.6 0.6) (drill 0.33) (layers *.Cu *.Mask)
-      (net 3 GND) (zone_connect 1))
-    (pad 2 thru_hole circle (at -1.27 -18.415 180) (size 0.6 0.6) (drill 0.33) (layers *.Cu *.Mask)
-      (net 3 GND) (zone_connect 1))
-    (pad 2 thru_hole circle (at 0 -18.415 180) (size 0.6 0.6) (drill 0.33) (layers *.Cu *.Mask)
-      (net 3 GND) (zone_connect 1))
-    (pad 2 thru_hole circle (at 1.27 -18.415 180) (size 0.6 0.6) (drill 0.33) (layers *.Cu *.Mask)
-      (net 3 GND) (zone_connect 1))
-    (pad 2 thru_hole circle (at 2.54 -18.415 180) (size 0.6 0.6) (drill 0.33) (layers *.Cu *.Mask)
-      (net 3 GND) (zone_connect 1))
-    (pad 2 thru_hole circle (at 3.175 -17.145 180) (size 0.6 0.6) (drill 0.33) (layers *.Cu *.Mask)
-      (net 3 GND) (zone_connect 1))
-    (pad 2 thru_hole circle (at 3.175 -15.875 180) (size 0.6 0.6) (drill 0.33) (layers *.Cu *.Mask)
-      (net 3 GND) (zone_connect 1))
-    (pad 2 thru_hole circle (at 3.175 -14.605 180) (size 0.6 0.6) (drill 0.33) (layers *.Cu *.Mask)
-      (net 3 GND) (zone_connect 1))
-    (pad 2 thru_hole circle (at 3.175 -13.335 180) (size 0.6 0.6) (drill 0.33) (layers *.Cu *.Mask)
-      (net 3 GND) (zone_connect 1))
-    (pad 1 thru_hole circle (at -2.54 0 180) (size 1.8 1.8) (drill 0.8) (layers *.Cu *.Mask)
-      (net 5 VDD))
-    (pad 2 thru_hole circle (at 0 0 180) (size 1.8 1.8) (drill 0.8) (layers *.Cu *.Mask)
-      (net 3 GND))
-    (pad 3 thru_hole circle (at 2.54 0 180) (size 1.8 1.8) (drill 0.8) (layers *.Cu *.Mask)
-      (net 1 +5V))
-  )
   (module Connectors_Terminal_Blocks:TerminalBlock_Pheonix_PT-3.5mm_4pol (layer F.Cu)
     (at 197.25 92.5 180)
@@
       (net 7 8A))
     (pad ~ thru_hole circle (at 4.34 -2.75) (size 1.75 1.75) (drill 1.5) (layers *.Cu *.Mask))
+  )
+  (module MDB_footprints:7805-thermal-conn (layer F.Cu)
+    (at 193.04 105.41 180)
+    (fp_text reference VREG (at 0 2.6 180) (layer F.SilkS)
+      (effects (font (size 1.2 1.2) (thickness 0.15)))
+    )
+    (fp_text value 7805 (at 0 -20.32 180) (layer F.Fab)
+      (effects (font (size 1.2 1.2) (thickness 0.15)))
+    )
+    (fp_line (start 3.94 -1.4) (end -3.94 -1.4) (layer F.SilkS) (width 0.15))
+    (fp_line (start -3.94 -19) (end 3.94 -19) (layer F.SilkS) (width 0.15))
+    (fp_line (start 3.94 -19) (end 3.94 1.4) (layer F.SilkS) (width 0.15))
+    (fp_line (start 3.94 1.4) (end -3.94 1.4) (layer F.SilkS) (width 0.15))
+    (fp_line (start -3.94 1.4) (end -3.94 -19) (layer F.SilkS) (width 0.15))
+    (fp_line (start -1.27 -1.4) (end -1.27 1.4) (layer F.SilkS) (width 0.15))
+    (pad 2 thru_hole circle (at -3.175 -13.335 180) (size 0.6 0.6) (drill 0.33) (layers *.Cu *.Mask)
+      (net 3 GND) (zone_connect 1))
+    (pad 2 thru_hole circle (at -3.175 -14.605 180) (size 0.6 0.6) (drill 0.33) (layers *.Cu *.Mask)
+      (net 3 GND) (zone_connect 1))
+    (pad 2 thru_hole circle (at -3.175 -15.875 180) (size 0.6 0.6) (drill 0.33) (layers *.Cu *.Mask)
+      (net 3 GND) (zone_connect 1))
+    (pad 2 thru_hole circle (at -3.175 -17.145 180) (size 0.6 0.6) (drill 0.33) (layers *.Cu *.Mask)
+      (net 3 GND) (zone_connect 1))
+    (pad 2 thru_hole circle (at -2.54 -18.415 180) (size 0.6 0.6) (drill 0.33) (layers *.Cu *.Mask)
+      (net 3 GND) (zone_connect 1))
+    (pad 2 thru_hole circle (at -1.27 -18.415 180) (size 0.6 0.6) (drill 0.33) (layers *.Cu *.Mask)
+      (net 3 GND) (zone_connect 1))
+    (pad 2 thru_hole circle (at 0 -18.415 180) (size 0.6 0.6) (drill 0.33) (layers *.Cu *.Mask)
+      (net 3 GND) (zone_connect 1))
+    (pad 2 thru_hole circle (at 1.27 -18.415 180) (size 0.6 0.6) (drill 0.33) (layers *.Cu *.Mask)
+      (net 3 GND) (zone_connect 1))
+    (pad 2 thru_hole circle (at 2.54 -18.415 180) (size 0.6 0.6) (drill 0.33) (layers *.Cu *.Mask)
+      (net 3 GND) (zone_connect 1))
+    (pad 2 thru_hole circle (at 3.175 -17.145 180) (size 0.6 0.6) (drill 0.33) (layers *.Cu *.Mask)
+      (net 3 GND) (zone_connect 1))
+    (pad 2 thru_hole circle (at 3.175 -15.875 180) (size 0.6 0.6) (drill 0.33) (layers *.Cu *.Mask)
+      (net 3 GND) (zone_connect 1))
+    (pad 2 thru_hole circle (at 3.175 -14.605 180) (size 0.6 0.6) (drill 0.33) (layers *.Cu *.Mask)
+      (net 3 GND) (zone_connect 1))
+    (pad 2 thru_hole circle (at 3.175 -13.335 180) (size 0.6 0.6) (drill 0.33) (layers *.Cu *.Mask)
+      (net 3 GND) (zone_connect 1))
+    (pad 1 thru_hole circle (at -2.54 0 180) (size 1.8 1.8) (drill 0.8) (layers *.Cu *.Mask)
+      (net 5 VDD))
+    (pad 2 thru_hole circle (at 0 0 180) (size 1.8 1.8) (drill 0.8) (layers *.Cu *.Mask)
+      (net 3 GND))
+    (pad 3 thru_hole circle (at 2.54 0 180) (size 1.8 1.8) (drill 0.8) (layers *.Cu *.Mask)
+      (net 1 +5V))
+    (pad 2 thru_hole rect (at 0 -15.24 180) (size 5 5) (drill 1) (layers *.Cu *.Mask)
+      (net 3 GND))
   )
   (gr_text "C. McElroy 19" (at 187.325 120.015 90) (layer F.SilkS)
@@
   (via (at 202.565 116.84) (size 0.6) (drill 0.4) (layers F.Cu B.Cu) (net 6))
   (segment (start 202.565 135.89) (end 202.565 116.84) (width 0.51) (layer F.Cu) (net 6))
-  (segment (start 212.725 96.52) (end 208.915 92.71) (width 0.51) (layer F.Cu) (net 6) (status 800000))
+  (segment (start 212.725 96.52) (end 208.915 92.71) (width 0.51) (layer F.Cu) (net 6))
   (segment (start 202.565 106.68) (end 212.725 96.52) (width 0.51) (layer F.Cu) (net 6))
-  (segment (start 208.915 92.71) (end 208.28 92.71) (width 0.51) (layer F.Cu) (net 6) (status C00000))
+  (segment (start 208.915 92.71) (end 208.28 92.71) (width 0.51) (layer F.Cu) (net 6))
   (segment (start 214.63 137.795) (end 214.63 96.52) (width 0.51) (layer F.Cu) (net 7))
   (segment (start 212.09 140.335) (end 214.63 137.795) (width 0.51) (layer F.Cu) (net 7))
@@
       )
     )
-  )
-  (zone (net 3) (net_name GND) (layer F.Cu) (hatch edge 0.508)
-    (connect_pads (clearance 0.3))
-    (min_thickness 0.254)
-    (fill yes (arc_segments 16) (thermal_gap 0.508) (thermal_bridge_width 0.508))
-    (polygon
-      (pts
-        (xy 189.23 117.475) (xy 196.85 117.475) (xy 196.85 124.46) (xy 189.23 124.46)
-      )
-    )
