File: MTB/MTB.sch (KiCad schematic (older format))
At the start: 45 parts, among them J1 BAT_CONN

Commit message: finished motherboard
Parts:
- removed B2: Buffer, Housings_DIP:DIP-14_W7.62mm_Socket, symbol Buffer
- added B2: Buffer2, Housings_DIP:DIP-14_W7.62mm_Socket, symbol Buffer2
- added T1, T2: TEST_HOLE, MCB_footprints:TESTPOINT_LARGE, symbol TEST_HOLE
- F1: value 2.0A Fuse -> .35A Fuse; footprint Capacitors_THT:C_Disc_D7.0mm_W2.5mm_P5.00mm -> MTB_footprints:1206
- F2: value 0.35A Fuse -> .35A Fuse
- F3: value 0.5A Fuse -> .5A Fuse
- F4: value 0.35A Fuse -> 2.0A Fuse; footprint MTB_footprints:1206 -> Capacitors_THT:C_Disc_D7.0mm_W2.5mm_P5.00mm
- PTB1: footprint Pin_Headers:Pin_Header_Straight_2x07 -> MTB_footprints:PTB_CONN
- renumbered C2 to C1, C1 to C2, C4 to C3, C3 to C4, C6 to C5, C5 to C6
Connections:
- net 2A: now also B2.8 (4Y)
- net 2AT: now also B2.9 (4A)
- net 4A: now also B2.11 (3Y)
- net 4AT: now also B2.12 (3A)
- net 6A: now also B2.3 (2Y)
- net 6AT: now also B2.2 (2A)
- net 8A: now also B2.6 (1Y)
- net 8AT: now also B2.5 (1A)
- net GND: now also B2.1 (2ŌĒ), B2.10 (4ŌĒ), B2.13 (3ŌĒ), B2.4 (1ŌĒ), B2.7 (GND), T1.1, T2.1
- net Vd: now also B1.14 (Vcc), C3.1, VR2.2 (VO), B2.14 (Vcc); no longer C5.1, VR3.2 (VO)
- net Vt: now also C5.1, VR3.2 (VO); no longer B1.14 (Vcc), C3.1, VR2.2 (VO)
- net at F1.2: now also C2.1, VR1.3 (VI); no longer MCB1.3 (trial)
- net at C4.1, VR2.3 (VI): now also F2.2; no longer F3.2
- net at C6.1, VR3.3 (VI): now also F3.2; no longer F4.2
- new net Vm: F4.2, MCB1.3 (trial)
Other:
- moved on the sheet: B1
