File: MTB/MTB.kicad_pcb (KiCad board)
At the start: 2 copper layers, 45 parts, among them J1 BAT_CONN

Commit message: finished motherboard
Parts:
- removed F4: 0.35A Fuse, MTB_footprints:1206
- removed PTB1: Protoboard, Pin_Headers:Pin_Header_Straight_2x07
- removed VR1: 5V_Regulator, MTB_footprints:VREG
- removed VR2, VR3: 3.3V_Regulator, MTB_footprints:VREG
- added 2.0A Fuse: 2.0A Fuse, Capacitors_THT:C_Disc_D7.0mm_W2.5mm_P5.00mm, F.Cu at (215.9, 83.8)
- added 3.3V Regulator: 3.3V_Regulator, MTB_footprints:VREG, F.Cu at (193.0, 114.3)
- added 3.3V Regulator: 3.3V_Regulator, MTB_footprints:VREG, F.Cu at (200.7, 127.0)
- added 5V Regulator: 5V_Regulator, MTB_footprints:VREG, F.Cu at (208.3, 94.0)
- added Protoboard: Protoboard, MTB_footprints:PTB_CONN, F.Cu at (124.5, 99.1)
- added T1: TEST_HOLE, MCB_footprints:TESTPOINT_LARGE, F.Cu at (120.7, 67.3)
- added T2: TEST_HOLE, MCB_footprints:TESTPOINT_LARGE, F.Cu at (120.7, 143.5)
- BATTERY LOW: renamed from LED5
- Buffer: renamed from B2; value Buffer -> Buffer2
- F1: value 2.0A Fuse -> .35A Fuse; footprint Capacitors_THT:C_Disc_D7.0mm_W2.5mm_P5.00mm -> MTB_footprints:1206
- F2: value 0.35A Fuse -> .35A Fuse
- F3: value 0.5A Fuse -> .5A Fuse
- Motor Control Board: renamed from MCB1
- moved D6 62.6 mm to (138.4, 105.4)
- moved D1 62.3 mm to (138.4, 111.8)
- moved D5 53.7 mm to (144.8, 105.4)
- moved D2 53.6 mm to (144.8, 111.8)
- moved C1 52.3 mm to (209.6, 88.9), turned to 180 degrees
- moved D4 51.5 mm to (151.1, 105.4)
- moved C5 47.7 mm to (205.7, 129.5), turned to 90 degrees
- moved D3 47.6 mm to (151.1, 111.8)
- moved C2 45.5 mm to (204.5, 88.9)
- moved C6 44.4 mm to (205.7, 124.5), turned to 270 degrees
- moved J1 41.9 mm to (215.9, 127.0), turned to 270 degrees
- moved Buffer 40.7 mm to (198.1, 78.7)
- moved C4 35.9 mm to (195.6, 118.1), turned to 180 degrees
- moved C3 32.5 mm to (190.5, 118.1)
- moved F2 31.5 mm to (210.8, 118.1), turned to 180 degrees
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- renumbered B1 to Buffer, COM1 to COMP, GPS1 to GPS, LED3 to GPS, IMU1 to IMU, LED2 to IMU, LED1 to SD, LED4 to TSY, TSY1 to Teensy-LC, SD1 to microSD
Connections:
- Buffer pad 14: Vt -> Vd (x2)
- Buffer pad 11: /2A -> /4A
- Buffer pad 12: 2AT -> 4AT
- Buffer pad 2: 8AT -> 6AT
- Buffer pad 3: /8A -> /6A
- Buffer pad 5: 6AT -> 8AT
- Buffer pad 6: /6A -> /8A
- Buffer pad 8: /4A -> /2A
- Buffer pad 9: 4AT -> 2AT
- C1 pad 1: Net-(C1-Pad1) -> +5V
- C2 pad 1: +5V -> Net-(C2-Pad1)
- C3 pad 1: Net-(C3-Pad1) -> Vd
- C4 pad 1: Vt -> Net-(C4-Pad1)
- C5 pad 1: Net-(C5-Pad1) -> Vt
- C6 pad 1: Vd -> Net-(C6-Pad1)
- F1 pad 1: Vm -> Vb
- F1 pad 2: Net-(F1-Pad2) -> Net-(C2-Pad1)
- F2 pad 1: Vm -> Vb
- F2 pad 2: Net-(C1-Pad1) -> Net-(C4-Pad1)
- F3 pad 1: Vm -> Vb
- F3 pad 2: Net-(C3-Pad1) -> Net-(C6-Pad1)
- J1 pad 1: Vm -> Vb
- Motor Control Board pad 3: Net-(F1-Pad2) -> Vm
- R6 pad 2: Vm -> Vb
Routing:
- net Vb: track 0.00 -> 298.3 mm, vias 0 -> 4
- net SDA0: track 0.00 -> 126.5 mm, vias 0 -> 4
- net D5: track 0.00 -> 122.0 mm, vias 0 -> 2
- net A0: track 0.00 -> 117.0 mm, vias 0 -> 7
- net RX: track 0.00 -> 108.5 mm, vias 0 -> 7
- net Vd: track 0.00 -> 93.2 mm, vias 0 -> 7
- net A1: track 0.00 -> 92.7 mm, vias 0 -> 4
- net 6AT: track 0.00 -> 88.4 mm
- net SCK0: track 0.00 -> 86.4 mm, vias 0 -> 6
- net CS0: track 0.00 -> 83.7 mm, vias 0 -> 2
- net D7: track 0.00 -> 82.1 mm, vias 0 -> 3
- net 8AT: track 0.00 -> 79.6 mm
- net 2AT: track 0.00 -> 79.3 mm, vias 0 -> 2
- net MISO0: track 0.00 -> 79.0 mm, vias 0 -> 2
- net MOSI0: track 0.00 -> 77.1 mm, vias 0 -> 7
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- added copper zone on In2.Cu, net +5V
- added copper zone on In1.Cu, net GND
- added copper zone on In2.Cu, net Vd
- added copper zone on In2.Cu, net Vt
Other:
- board outline added: 101.6 x 83.8 mm
- copper layers 2 -> 4
- net class Default: trace_width 0.25 -> 0.5
- net class High Power added: clearance 0.2, trace_width 1.9, via_dia 0.6, via_drill 0.4
- net class Power added: clearance 0.2, trace_width 1.27, via_dia 0.6, via_drill 0.4
- board text added: "(buffered)"
- board text added: "0.1µF"
- board text added: "1.0µF"
- board text added: "1A"
- board text added: "2A"
- board text added: "3A"
- board text added: "4A"
- board text added: "5A"
- board text added: "5V"
- board text added: "6A"
- board text added: "7A"
- board text added: "8A"
- board text added: "A0"
- board text added: "A1"
- board text added: "A10"
- board text added: "A11"
- board text added: "A12"
- board text added: "A7"
- board text added: "A9"
- board text added: "CS"
- board text added: "D5"
- board text added: "D7"
- board text added: "D8"
- board text added: "Diode Clamps"
- board text added: "E80 Motherboard V2.0"
- board text added: "GND"
- board text added: "MISO"
- board text added: "MOSI"
- board text added: "RX"
- board text added: "S1"
- board text added: "SCK"
- board text added: "SCL"
- board text added: "SDA"
- board text added: "TX"
- board text added: "Vb"
- board text added: "Vd"
- board text added: "Vm"
- board text added: "Vt"
- board text added: "for Diode Clamps Buffers"
- board text added: "for GPS MCB"
- board text added: "for Teensy IMU SD Battery Monitor"

Commit message: small mtb updates
Routing:
- net Vm: track 41.8 -> 40.7 mm
Other:
- board text added: "Black"
- board text added: "C. McElroy 19"
- board text added: "Red"
Changed lines of the file:
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@@
     (area 111.034999 62.525 219.775 148.395)
     (thickness 1.6)
-    (drawings 152)
-    (tracks 609)
+    (drawings 155)
+    (tracks 611)
     (zones 0)
     (modules 47)
@@
     (pad_to_mask_clearance 0.2)
     (aux_axis_origin 0 0)
-    (visible_elements FFFEF77F)
+    (visible_elements FFFEFF7F)
     (pcbplotparams
-      (layerselection 0x00030_80000001)
+      (layerselection 0x010f0_80000007)
       (usegerberextensions false)
       (excludeedgelayer true)
@@
       (outputformat 1)
       (mirror false)
-      (drillshape 1)
+      (drillshape 0)
       (scaleselection 1)
-      (outputdirectory ""))
+      (outputdirectory MTB_plot/))
   )
   (net 0 "")
@@
     (pad 36 thru_hole circle (at 33.02 -2.54) (size 1.524 1.524) (drill 0.762) (layers *.Cu *.Mask))
   )
+  (gr_text "C. McElroy 19" (at 131.318 144.272) (layer F.SilkS)
+    (effects (font (size 1 1) (thickness 0.15)))
+  )
+  (gr_text Red (at 212.598 123.952) (layer F.SilkS)
+    (effects (font (size 1 1) (thickness 0.15)))
+  )
+  (gr_text Black (at 211.455 130.81) (layer F.SilkS)
+    (effects (font (size 1 1) (thickness 0.15)))
+  )
   (gr_text "E80 Motherboard V2.0" (at 138.43 142.24) (layer F.SilkS)
     (effects (font (size 1.5 1.5) (thickness 0.3)))
@@
   (gr_line (start 218.44 147.32) (end 116.84 147.32) (angle 90) (layer Edge.Cuts) (width 0.15))
   (gr_line (start 218.44 63.5) (end 218.44 147.32) (angle 90) (layer Edge.Cuts) (width 0.15))
-  (segment (start 199.39 74.168) (end 198.882 74.93) (width 0.89) (layer F.Cu) (net 0))
-  (segment (start 192.278 74.93) (end 194.056 75.946) (width 0.89) (layer F.Cu) (net 0))
-  (segment (start 194.056 75.946) (end 195.58 76.2) (width 0.89) (layer F.Cu) (net 0))
-  (segment (start 195.58 76.2) (end 197.104 75.946) (width 0.89) (layer F.Cu) (net 0))
-  (segment (start 197.104 75.946) (end 198.882 74.93) (width 0.89) (layer F.Cu) (net 0))
-  (segment (start 191.77 74.168) (end 192.278 74.93) (width 0.89) (layer F.Cu) (net 0))
-  (segment (start 194.31 71.12) (end 194.1576 70.8152) (width 0.89) (layer F.Cu) (net 0))
-  (segment (start 191.96304 70.78472) (end 191.77 71.12) (width 0.89) (layer F.Cu) (net 0))
-  (segment (start 192.532 70.358) (end 191.96304 70.78472) (width 0.89) (layer F.Cu) (net 0))
-  (segment (start 193.02984 70.28688) (end 192.532 70.358) (width 0.89) (layer F.Cu) (net 0))
-  (segment (start 193.548 70.358) (end 193.02984 70.28688) (width 0.89) (layer F.Cu) (net 0))
-  (segment (start 194.1576 70.8152) (end 193.548 70.358) (width 0.89) (layer F.Cu) (net 0))
-  (segment (start 199.39 71.12) (end 196.85 71.12) (width 0.89) (layer F.Cu) (net 0))
+  (segment (start 134.62 77.978) (end 134.112 78.74) (width 0.89) (layer F.Cu) (net 0))
+  (segment (start 127.508 78.74) (end 129.286 79.756) (width 0.89) (layer F.Cu) (net 0))
+  (segment (start 129.286 79.756) (end 130.81 80.01) (width 0.89) (layer F.Cu) (net 0))
+  (segment (start 130.81 80.01) (end 132.334 79.756) (width 0.89) (layer F.Cu) (net 0))
+  (segment (start 132.334 79.756) (end 134.112 78.74) (width 0.89) (layer F.Cu) (net 0))
+  (segment (start 127 77.978) (end 127.508 78.74) (width 0.89) (layer F.Cu) (net 0))
+  (segment (start 129.54 74.93) (end 129.3876 74.6252) (width 0.89) (layer F.Cu) (net 0))
+  (segment (start 127.19304 74.59472) (end 127 74.93) (width 0.89) (layer F.Cu) (net 0))
+  (segment (start 127.762 74.168) (end 127.19304 74.59472) (width 0.89) (layer F.Cu) (net 0))
+  (segment (start 128.25984 74.09688) (end 127.762 74.168) (width 0.89) (layer F.Cu) (net 0))
+  (segment (start 128.778 74.168) (end 128.25984 74.09688) (width 0.89) (layer F.Cu) (net 0))
+  (segment (start 129.3876 74.6252) (end 128.778 74.168) (width 0.89) (layer F.Cu) (net 0))
+  (segment (start 134.62 74.93) (end 132.08 74.93) (width 0.89) (layer F.Cu) (net 0))
   (segment (start 165.1 142.748) (end 165.1 145.415) (width 1.9) (layer F.Cu) (net 1))
   (via (at 165.1 145.415) (size 0.6) (drill 0.4) (layers F.Cu B.Cu) (net 1))
@@
   (segment (start 127 101.6) (end 129.54 99.06) (width 1.27) (layer In2.Cu) (net 35))
   (segment (start 127 116.84) (end 128.27 118.11) (width 1.27) (layer In2.Cu) (net 35))
-  (segment (start 200.66 91.44) (end 175.26 91.44) (width 1.9) (layer In2.Cu) (net 36) (status 20))
-  (segment (start 200.66 86.36) (end 200.66 91.44) (width 1.9) (layer In2.Cu) (net 36))
+  (segment (start 200.66 89.535) (end 181.61 89.535) (width 1.9) (layer In2.Cu) (net 36))
+  (segment (start 210.9 83.82) (end 203.2 83.82) (width 1.9) (layer In2.Cu) (net 36))
   (segment (start 203.2 83.82) (end 200.66 86.36) (width 1.9) (layer In2.Cu) (net 36))
-  (segment (start 210.9 83.82) (end 203.2 83.82) (width 1.9) (layer In2.Cu) (net 36))
+  (segment (start 200.66 86.36) (end 200.66 89.535) (width 1.9) (layer In2.Cu) (net 36))
+  (segment (start 179.705 91.44) (end 175.26 91.44) (width 1.9) (layer In2.Cu) (net 36) (status 800000))
+  (segment (start 181.61 89.535) (end 179.705 91.44) (width 1.9) (layer In2.Cu) (net 36))
   (segment (start 132.08 114.3) (end 132.08 116.84) (width 0.5) (layer B.Cu) (net 37))
   (segment (start 180.455 137.68) (end 181.61 137.68) (width 0.5) (layer F.Cu) (net 37))
@@
   (via (at 212.344 143.002) (size 0.6) (drill 0.4) (layers F.Cu B.Cu) (net 45))
   (segment (start 212.344 143.002) (end 212.346 143) (width 0.5) (layer F.Cu) (net 45))
-  (segment (start 214.255 143) (end 212.346 143) (width 0.5) (layer F.Cu) (net 45) (status 400000))
+  (segment (start 214.255 143) (end 212.346 143) (width 0.5) (layer F.Cu) (net 45))
   (segment (start 169.545 114.3) (end 162.56 114.3) (width 0.5) (layer F.Cu) (net 45))
   (segment (start 190.5 135.255) (end 193.801863 132.085904) (width 0.5) (layer F.Cu) (net 45))
@@
   (via (at 175.26 111.76) (size 0.6) (drill 0.4) (layers F.Cu B.Cu) (net 46))
   (segment (start 175.26 111.76) (end 175.26 118.11) (width 0.5) (layer F.Cu) (net 46))
-  (segment (start 212.514 140.8) (end 214.255 140.8) (width 0.5) (layer F.Cu) (net 46) (status 800000))
+  (segment (start 212.514 140.8) (end 214.255 140.8) (width 0.5) (layer F.Cu) (net 46))
   (segment (start 212.344 140.97) (end 212.514 140.8) (width 0.5) (layer F.Cu) (net 46))
   (via (at 212.344 140.97) (size 0.6) (drill 0.4) (layers F.Cu B.Cu) (net 46))
@@
   (segment (start 157.48 115.062) (end 150.368 122.174) (width 0.5) (layer F.Cu) (net 47))
   (segment (start 202.946 137.414) (end 200.025 140.335) (width 0.5) (layer B.Cu) (net 47))
-  (segment (start 212.43 137.5) (end 214.255 137.5) (width 0.5) (layer F.Cu) (net 47) (status 800000))
+  (segment (start 212.43 137.5) (end 214.255 137.5) (width 0.5) (layer F.Cu) (net 47))
   (segment (start 212.344 137.414) (end 212.43 137.5) (width 0.5) (layer F.Cu) (net 47))
   (via (at 212.344 137.414) (size 0.6) (drill 0.4) (layers F.Cu B.Cu) (net 47))
@@
     (polygon
       (pts
-        (xy 215.9 101.6) (xy 167.64 101.6) (xy 167.64 93.98) (xy 119.38 93.98) (xy 119.38 68.58)
+        (xy 214.63 102.235) (xy 166.37 102.235) (xy 167.64 93.98) (xy 119.38 93.98) (xy 119.38 68.58)
         (xy 215.9 68.58)
       )
@@
     (polygon
       (pts
-        (xy 200.66 104.14) (xy 200.66 120.65) (xy 130.81 120.65) (xy 130.81 102.87) (xy 165.1 102.87)
-        (xy 165.1 104.14)
+        (xy 200.66 104.14) (xy 200.66 120.65) (xy 130.81 120.65) (xy 130.81 102.87) (xy 163.83 102.87)
+        (xy 163.83 104.14)
       )
     )
